File: KiCad PCB Files/fret clone.kicad_sch (KiCad schematic)
At the start: 7 parts, among them J1 Conn_01x03_Pin, J2 Conn_01x03_Pin

Commit message: add the things new LED
Parts:
- added J3: Conn_01x04_Pin, Connector_PinHeader_2.54mm:PinHeader_1x04_P2.54mm_Vertical, symbol Connector:Conn_01x04_Pin
- added LED1, LED2, LED3, LED4, LED5: ~, sk9822-ec20:SK9822-EC20, symbol sk9822-ec20-2:SK9822-EC20
- CH1, CH2, CH3, CH4, CH5: footprint PCM_Switch_Keyboard_Kailh:SW_Kailh_Choc_Mini_1.00u -> PCM_Switch_Keyboard_Kailh:SW_Kailh_Choc_Mini
Connections:
- new net: LED2.1 (SDO), LED3.3 (SDI)
- new net: LED1.1 (SDO), LED2.3 (SDI)
- new net: LED1.6 (CKO), LED2.4 (CKI)
- new net: J3.3 (Pin_3), LED1.5 (VDD), LED2.5 (VDD), LED3.5 (VDD), LED4.5 (VDD), LED5.5 (VDD)
- new net: LED2.6 (CKO), LED3.4 (CKI)
- new net: LED3.1 (SDO), LED4.3 (SDI)
- new net: LED3.6 (CKO), LED4.4 (CKI)
- new net: J3.1 (Pin_1), LED1.3 (SDI)
- new net: J3.2 (Pin_2), LED1.4 (CKI)
- new net: LED4.1 (SDO), LED5.3 (SDI)
- new net: LED4.6 (CKO), LED5.4 (CKI)
- new net GND: J3.4 (Pin_4), LED1.2 (GND), LED2.2 (GND), LED3.2 (GND), LED4.2 (GND), LED5.2 (GND)
